File: hardware/microProc/Power_supply.kicad_sch (KiCad schematic)
At the start: 0 parts

Commit message: Ajout de la feuille Power supply
Signed-off-by: Martin RYS <martinrys@sfr.fr>
Parts:
- added C? (x2): 1uF, symbol Device:C
- added D?: LED, symbol Device:LED
- added R?: 1k, symbol Device:R
- added U?: BU33SD5WG-TR, Package_TO_SOT_SMD:SOT-23-5, symbol Regulator_Linear:MCP1802x-xx02xOT
Connections:
- new net: D?.1 (K), R?.1
- new net +3V3: C?.1, D?.2 (A), U?.5 (VOUT)
- new net +5V: C?.1, U?.1 (VIN), U?.3 (~{SHDN})
- new net GND: C?.2, C?.2, R?.2, U?.2 (GND)
Changed lines of the file:
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@@
 (kicad_sch (version 20211123) (generator eeschema)
   (paper "A4")
+  (junction (at 135.89 77.47) (diameter 0) (color 0 0 0 0)
+  )
+  (junction (at 125.73 87.63) (diameter 0) (color 0 0 0 0)
+  )
+  (junction (at 125.73 77.47) (diameter 0) (color 0 0 0 0)
+  )
+  (junction (at 146.05 87.63) (diameter 0) (color 0 0 0 0)
+  )
+  (junction (at 165.1 77.47) (diameter 0) (color 0 0 0 0)
+  )
+  (wire (pts (xy 185.42 74.93) (xy 185.42 78.74))
+    (stroke (width 0) (type default) (color 0 0 0 0))
+  )
+  (wire (pts (xy 135.89 77.47) (xy 125.73 77.47))
+    (stroke (width 0) (type default) (color 0 0 0 0))
+  )
+  (wire (pts (xy 165.1 77.47) (xy 156.21 77.47))
+    (stroke (width 0) (type default) (color 0 0 0 0))
+  )
+  (wire (pts (xy 125.73 87.63) (xy 146.05 87.63))
+    (stroke (width 0) (type default) (color 0 0 0 0))
+  )
+  (wire (pts (xy 125.73 85.09) (xy 125.73 87.63))
+    (stroke (width 0) (type default) (color 0 0 0 0))
+  )
+  (wire (pts (xy 185.42 86.36) (xy 185.42 87.63))
+    (stroke (width 0) (type default) (color 0 0 0 0))
+  )
+  (wire (pts (xy 146.05 87.63) (xy 165.1 87.63))
+    (stroke (width 0) (type default) (color 0 0 0 0))
+  )
+  (wire (pts (xy 165.1 87.63) (xy 165.1 86.36))
+    (stroke (width 0) (type default) (color 0 0 0 0))
+  )
+  (wire (pts (xy 135.89 80.01) (xy 135.89 77.47))
+    (stroke (width 0) (type default) (color 0 0 0 0))
+  )
+  (wire (pts (xy 165.1 78.74) (xy 165.1 77.47))
+    (stroke (width 0) (type default) (color 0 0 0 0))
+  )
+  (symbol (lib_id "Device:LED") (at 185.42 71.12 90) (unit 1)
+    (in_bom yes) (on_board yes) (fields_autoplaced)
+    (property "Reference" "D?" (id 0) (at 189.23 71.4374 90)
+      (effects (font (size 1.27 1.27)) (justify right))
+    )
+    (property "Value" "LED" (id 1) (at 189.23 73.9774 90)
+      (effects (font (size 1.27 1.27)) (justify right))
+    )
+    (property "Footprint" "" (id 2) (at 185.42 71.12 0)
+      (effects (font (size 1.27 1.27)) hide)
+    )
+    (property "Datasheet" "~" (id 3) (at 185.42 71.12 0)
+      (effects (font (size 1.27 1.27)) hide)
+    )
+    (pin "1")
+    (pin "2")
+  )
+  (symbol (lib_id "power:+3V3") (at 185.42 67.31 0) (unit 1)
+    (in_bom yes) (on_board yes) (fields_autoplaced)
+    (property "Reference" "#PWR?" (id 0) (at 185.42 71.12 0)
+      (effects (font (size 1.27 1.27)) hide)
+    )
+    (property "Value" "+3V3" (id 1) (at 185.42 62.23 0))
+    (property "Footprint" "" (id 2) (at 185.42 67.31 0)
+      (effects (font (size 1.27 1.27)) hide)
+    )
+    (property "Datasheet" "" (id 3) (at 185.42 67.31 0)
+      (effects (font (size 1.27 1.27)) hide)
+    )
+    (pin "1")
+  )
+  (symbol (lib_id "power:+3V3") (at 165.1 77.47 0) (unit 1)
+    (in_bom yes) (on_board yes) (fields_autoplaced)
+    (property "Reference" "#PWR?" (id 0) (at 165.1 81.28 0)
+      (effects (font (size 1.27 1.27)) hide)
+    )
+    (property "Value" "+3V3" (id 1) (at 165.1 72.39 0))
+    (property "Footprint" "" (id 2) (at 165.1 77.47 0)
+      (effects (font (size 1.27 1.27)) hide)
+    )
+    (property "Datasheet" "" (id 3) (at 165.1 77.47 0)
+      (effects (font (size 1.27 1.27)) hide)
+    )
+    (pin "1")
+  )
+  (symbol (lib_id "power:+5V") (at 125.73 77.47 0) (unit 1)
+    (in_bom yes) (on_board yes) (fields_autoplaced)
+    (property "Reference" "#PWR?" (id 0) (at 125.73 81.28 0)
+      (effects (font (size 1.27 1.27)) hide)
+    )
+    (property "Value" "+5V" (id 1) (at 125.73 72.39 0))
+    (property "Footprint" "" (id 2) (at 125.73 77.47 0)
+      (effects (font (size 1.27 1.27)) hide)
+    )
+    (property "Datasheet" "" (id 3) (at 125.73 77.47 0)
+      (effects (font (size 1.27 1.27)) hide)
+    )
+    (pin "1")
+  )
+  (symbol (lib_id "power:GND") (at 185.42 87.63 0) (unit 1)
+    (in_bom yes) (on_board yes) (fields_autoplaced)
+    (property "Reference" "#PWR?" (id 0) (at 185.42 93.98 0)
+      (effects (font (size 1.27 1.27)) hide)
+    )
+    (property "Value" "GND" (id 1) (at 185.42 92.71 0))
+    (property "Footprint" "" (id 2) (at 185.42 87.63 0)
+      (effects (font (size 1.27 1.27)) hide)
+    )
+    (property "Datasheet" "" (id 3) (at 185.42 87.63 0)
+      (effects (font (size 1.27 1.27)) hide)
+    )
+    (pin "1")
+  )
+  (symbol (lib_id "Device:R") (at 185.42 82.55 0) (unit 1)
+    (in_bom yes) (on_board yes) (fields_autoplaced)
+    (property "Reference" "R?" (id 0) (at 187.96 81.2799 0)
+      (effects (font (size 1.27 1.27)) (justify left))
+    )
+    (property "Value" "1k" (id 1) (at 187.96 83.8199 0)
+      (effects (font (size 1.27 1.27)) (justify left))
+    )
+    (property "Footprint" "" (id 2) (at 183.642 82.55 90)
+      (effects (font (size 1.27 1.27)) hide)
+    )
+    (property "Datasheet" "~" (id 3) (at 185.42 82.55 0)
+      (effects (font (size 1.27 1.27)) hide)
+    )
+    (pin "1")
+    (pin "2")
+  )
+  (symbol (lib_id "Device:C") (at 165.1 82.55 0) (unit 1)
+    (in_bom yes) (on_board yes) (fields_autoplaced)
+    (property "Reference" "C?" (id 0) (at 168.91 81.2799 0)
+      (effects (font (size 1.27 1.27)) (justify left))
+    )
+    (property "Value" "1uF" (id 1) (at 168.91 83.8199 0)
+      (effects (font (size 1.27 1.27)) (justify left))
+    )
+    (property "Footprint" "" (id 2) (at 166.0652 86.36 0)
+      (effects (font (size 1.27 1.27)) hide)
+    )
+    (property "Datasheet" "~" (id 3) (at 165.1 82.55 0)
+      (effects (font (size 1.27 1.27)) hide)
+    )
+    (pin "1")
+    (pin "2")
+  )
+  (symbol (lib_id "Device:C") (at 125.73 81.28 0) (unit 1)
+    (in_bom yes) (on_board yes) (fields_autoplaced)
+    (property "Reference" "C?" (id 0) (at 129.54 80.0099 0)
+      (effects (font (size 1.27 1.27)) (justify left))
+    )
+    (property "Value" "1uF" (id 1) (at 129.54 82.5499 0)
+      (effects (font (size 1.27 1.27)) (justify left))
+    )
+    (property "Footprint" "" (id 2) (at 126.6952 85.09 0)
+      (effects (font (size 1.27 1.27)) hide)
+    )
+    (property "Datasheet" "~" (id 3) (at 125.73 81.28 0)
+      (effects (font (size 1.27 1.27)) hide)
+    )
+    (pin "1")
+    (pin "2")
+  )
+  (symbol (lib_id "power:GND") (at 125.73 87.63 0) (unit 1)
+    (in_bom yes) (on_board yes) (fields_autoplaced)
+    (property "Reference" "#PWR?" (id 0) (at 125.73 93.98 0)
+      (effects (font (size 1.27 1.27)) hide)
+    )
+    (property "Value" "GND" (id 1) (at 125.73 92.71 0))
+    (property "Footprint" "" (id 2) (at 125.73 87.63 0)
+      (effects (font (size 1.27 1.27)) hide)
+    )
+    (property "Datasheet" "" (id 3) (at 125.73 87.63 0)
+      (effects (font (size 1.27 1.27)) hide)
+    )
+    (pin "1")
+  )
+  (symbol (lib_id "Regulator_Linear:MCP1802x-xx02xOT") (at 146.05 80.01 0) (unit 1)
+    (in_bom yes) (on_board yes) (fields_autoplaced)
+    (property "Reference" "U?" (id 0) (at 146.05 69.85 0))
+    (property "Value" "BU33SD5WG-TR" (id 1) (at 146.05 72.39 0))
+    (property "Footprint" "Package_TO_SOT_SMD:SOT-23-5" (id 2) (at 139.7 71.12 0)
+      (effects (font (size 1.27 1.27) italic) (justify left) hide)
+    )
+    (property "Datasheet" "http://ww1.microchip.com/downloads/en/DeviceDoc/22053C.pdf" (id 3) (at 146.05 82.55 0)
+      (effects (font (size 1.27 1.27)) hide)
+    )
+    (pin "1")
+    (pin "2")
+    (pin "3")
+    (pin "4")
+    (pin "5")
+  )
+  (sheet_instances
+    (path "/" (page "1"))
+  )
+  (symbol_instances
+    (path "/070425be-5ccb-4e88-8c4c-e4baef794b8e"
+      (reference "#PWR?") (unit 1) (value "+3V3") (footprint "")
+    )
+    (path "/3fa75c28-cd45-4a64-8a75-f1e20f7b02e4"
+      (reference "#PWR?") (unit 1) (value "+3V3") (footprint "")
+    )
+    (path "/44d6556c-3980-4535-91e7-ca0f03731d28"
+      (reference "#PWR?") (unit 1) (value "+5V") (footprint "")
+    )
+    (path "/52992af0-bfca-4eff-8f47-ab566d86e29d"
+      (reference "#PWR?") (unit 1) (value "GND") (footprint "")
+    )
+    (path "/d7482a1f-d519-46fd-95ed-f3094f05d90f"
+      (reference "#PWR?") (unit 1) (value "GND") (footprint "")
+    )
+    (path "/96102620-adf7-478e-bad6-78de1078c047"
+      (reference "C?") (unit 1) (value "1uF") (footprint "")
+    )
+    (path "/bcc8b894-fc6c-4a02-b892-9bb6d6a25acb"
+      (reference "C?") (unit 1) (value "1uF") (footprint "")
+    )
+    (path "/0220e075-d97f-4076-83a4-7e5c155e204a"
+      (reference "D?") (unit 1) (value "LED") (footprint "")
+    )
+    (path "/56bc323f-2c11-45f4-9795-9e890654428f"
+      (reference "R?") (unit 1) (value "1k") (footprint "")
+    )
+    (path "/eebe5061-3b92-49eb-a209-d76d8334c777"
+      (reference "U?") (unit 1) (value "BU33SD5WG-TR") (footprint "Package_TO_SOT_SMD:SOT-23-5")
+    )
+  )
 )

Commit message: SWD connector
Parts:
- removed C? (x2): 1uF, symbol Device:C
- removed D?: LED, symbol Device:LED
- removed R?: 1k, symbol Device:R
- removed U?: BU33SD5WG-TR, Package_TO_SOT_SMD:SOT-23-5, symbol Regulator_Linear:MCP1802x-xx02xOT
Changed lines of the file:
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@@
 (kicad_sch (version 20211123) (generator eeschema)
   (paper "A4")
-  (junction (at 135.89 77.47) (diameter 0) (color 0 0 0 0)
-  )
-  (junction (at 125.73 87.63) (diameter 0) (color 0 0 0 0)
-  )
-  (junction (at 125.73 77.47) (diameter 0) (color 0 0 0 0)
-  )
-  (junction (at 146.05 87.63) (diameter 0) (color 0 0 0 0)
-  )
-  (junction (at 165.1 77.47) (diameter 0) (color 0 0 0 0)
-  )
-  (wire (pts (xy 185.42 74.93) (xy 185.42 78.74))
-    (stroke (width 0) (type default) (color 0 0 0 0))
-  )
-  (wire (pts (xy 135.89 77.47) (xy 125.73 77.47))
-    (stroke (width 0) (type default) (color 0 0 0 0))
-  )
-  (wire (pts (xy 165.1 77.47) (xy 156.21 77.47))
-    (stroke (width 0) (type default) (color 0 0 0 0))
-  )
-  (wire (pts (xy 125.73 87.63) (xy 146.05 87.63))
-    (stroke (width 0) (type default) (color 0 0 0 0))
-  )
-  (wire (pts (xy 125.73 85.09) (xy 125.73 87.63))
-    (stroke (width 0) (type default) (color 0 0 0 0))
-  )
-  (wire (pts (xy 185.42 86.36) (xy 185.42 87.63))
-    (stroke (width 0) (type default) (color 0 0 0 0))
-  )
-  (wire (pts (xy 146.05 87.63) (xy 165.1 87.63))
-    (stroke (width 0) (type default) (color 0 0 0 0))
-  )
-  (wire (pts (xy 165.1 87.63) (xy 165.1 86.36))
-    (stroke (width 0) (type default) (color 0 0 0 0))
-  )
-  (wire (pts (xy 135.89 80.01) (xy 135.89 77.47))
-    (stroke (width 0) (type default) (color 0 0 0 0))
-  )
-  (wire (pts (xy 165.1 78.74) (xy 165.1 77.47))
-    (stroke (width 0) (type default) (color 0 0 0 0))
-  )
-  (symbol (lib_id "Device:LED") (at 185.42 71.12 90) (unit 1)
-    (in_bom yes) (on_board yes) (fields_autoplaced)
-    (property "Reference" "D?" (id 0) (at 189.23 71.4374 90)
-      (effects (font (size 1.27 1.27)) (justify right))
-    )
-    (property "Value" "LED" (id 1) (at 189.23 73.9774 90)
-      (effects (font (size 1.27 1.27)) (justify right))
-    )
-    (property "Footprint" "" (id 2) (at 185.42 71.12 0)
-      (effects (font (size 1.27 1.27)) hide)
-    )
-    (property "Datasheet" "~" (id 3) (at 185.42 71.12 0)
-      (effects (font (size 1.27 1.27)) hide)
-    )
-    (pin "1")
-    (pin "2")
-  )
-  (symbol (lib_id "power:+3V3") (at 185.42 67.31 0) (unit 1)
-    (in_bom yes) (on_board yes) (fields_autoplaced)
-    (property "Reference" "#PWR?" (id 0) (at 185.42 71.12 0)
-      (effects (font (size 1.27 1.27)) hide)
-    )
-    (property "Value" "+3V3" (id 1) (at 185.42 62.23 0))
-    (property "Footprint" "" (id 2) (at 185.42 67.31 0)
-      (effects (font (size 1.27 1.27)) hide)
-    )
-    (property "Datasheet" "" (id 3) (at 185.42 67.31 0)
-      (effects (font (size 1.27 1.27)) hide)
-    )
-    (pin "1")
-  )
-  (symbol (lib_id "power:+3V3") (at 165.1 77.47 0) (unit 1)
-    (in_bom yes) (on_board yes) (fields_autoplaced)
-    (property "Reference" "#PWR?" (id 0) (at 165.1 81.28 0)
-      (effects (font (size 1.27 1.27)) hide)
-    )
-    (property "Value" "+3V3" (id 1) (at 165.1 72.39 0))
-    (property "Footprint" "" (id 2) (at 165.1 77.47 0)
-      (effects (font (size 1.27 1.27)) hide)
-    )
-    (property "Datasheet" "" (id 3) (at 165.1 77.47 0)
-      (effects (font (size 1.27 1.27)) hide)
-    )
-    (pin "1")
-  )
-  (symbol (lib_id "power:+5V") (at 125.73 77.47 0) (unit 1)
-    (in_bom yes) (on_board yes) (fields_autoplaced)
-    (property "Reference" "#PWR?" (id 0) (at 125.73 81.28 0)
-      (effects (font (size 1.27 1.27)) hide)
-    )
-    (property "Value" "+5V" (id 1) (at 125.73 72.39 0))
-    (property "Footprint" "" (id 2) (at 125.73 77.47 0)
-      (effects (font (size 1.27 1.27)) hide)
-    )
-    (property "Datasheet" "" (id 3) (at 125.73 77.47 0)
-      (effects (font (size 1.27 1.27)) hide)
-    )
-    (pin "1")
-  )
-  (symbol (lib_id "power:GND") (at 185.42 87.63 0) (unit 1)
-    (in_bom yes) (on_board yes) (fields_autoplaced)
-    (property "Reference" "#PWR?" (id 0) (at 185.42 93.98 0)
-      (effects (font (size 1.27 1.27)) hide)
-    )
-    (property "Value" "GND" (id 1) (at 185.42 92.71 0))
-    (property "Footprint" "" (id 2) (at 185.42 87.63 0)
-      (effects (font (size 1.27 1.27)) hide)
-    )
-    (property "Datasheet" "" (id 3) (at 185.42 87.63 0)
-      (effects (font (size 1.27 1.27)) hide)
-    )
-    (pin "1")
-  )
-  (symbol (lib_id "Device:R") (at 185.42 82.55 0) (unit 1)
-    (in_bom yes) (on_board yes) (fields_autoplaced)
-    (property "Reference" "R?" (id 0) (at 187.96 81.2799 0)
-      (effects (font (size 1.27 1.27)) (justify left))
-    )
-    (property "Value" "1k" (id 1) (at 187.96 83.8199 0)
-      (effects (font (size 1.27 1.27)) (justify left))
-    )
-    (property "Footprint" "" (id 2) (at 183.642 82.55 90)
-      (effects (font (size 1.27 1.27)) hide)
-    )
-    (property "Datasheet" "~" (id 3) (at 185.42 82.55 0)
-      (effects (font (size 1.27 1.27)) hide)
-    )
-    (pin "1")
-    (pin "2")
-  )
-  (symbol (lib_id "Device:C") (at 165.1 82.55 0) (unit 1)
-    (in_bom yes) (on_board yes) (fields_autoplaced)
-    (property "Reference" "C?" (id 0) (at 168.91 81.2799 0)
-      (effects (font (size 1.27 1.27)) (justify left))
-    )
-    (property "Value" "1uF" (id 1) (at 168.91 83.8199 0)
-      (effects (font (size 1.27 1.27)) (justify left))
-    )
-    (property "Footprint" "" (id 2) (at 166.0652 86.36 0)
-      (effects (font (size 1.27 1.27)) hide)
-    )
-    (property "Datasheet" "~" (id 3) (at 165.1 82.55 0)
-      (effects (font (size 1.27 1.27)) hide)
-    )
-    (pin "1")
-    (pin "2")
-  )
-  (symbol (lib_id "Device:C") (at 125.73 81.28 0) (unit 1)
-    (in_bom yes) (on_board yes) (fields_autoplaced)
-    (property "Reference" "C?" (id 0) (at 129.54 80.0099 0)
-      (effects (font (size 1.27 1.27)) (justify left))
-    )
-    (property "Value" "1uF" (id 1) (at 129.54 82.5499 0)
-      (effects (font (size 1.27 1.27)) (justify left))
-    )
-    (property "Footprint" "" (id 2) (at 126.6952 85.09 0)
-      (effects (font (size 1.27 1.27)) hide)
-    )
-    (property "Datasheet" "~" (id 3) (at 125.73 81.28 0)
-      (effects (font (size 1.27 1.27)) hide)
-    )
-    (pin "1")
-    (pin "2")
-  )
-  (symbol (lib_id "power:GND") (at 125.73 87.63 0) (unit 1)
-    (in_bom yes) (on_board yes) (fields_autoplaced)
-    (property "Reference" "#PWR?" (id 0) (at 125.73 93.98 0)
-      (effects (font (size 1.27 1.27)) hide)
-    )
-    (property "Value" "GND" (id 1) (at 125.73 92.71 0))
-    (property "Footprint" "" (id 2) (at 125.73 87.63 0)
-      (effects (font (size 1.27 1.27)) hide)
-    )
-    (property "Datasheet" "" (id 3) (at 125.73 87.63 0)
-      (effects (font (size 1.27 1.27)) hide)
-    )
-    (pin "1")
-  )
-  (symbol (lib_id "Regulator_Linear:MCP1802x-xx02xOT") (at 146.05 80.01 0) (unit 1)
-    (in_bom yes) (on_board yes) (fields_autoplaced)
-    (property "Reference" "U?" (id 0) (at 146.05 69.85 0))
-    (property "Value" "BU33SD5WG-TR" (id 1) (at 146.05 72.39 0))
-    (property "Footprint" "Package_TO_SOT_SMD:SOT-23-5" (id 2) (at 139.7 71.12 0)
-      (effects (font (size 1.27 1.27) italic) (justify left) hide)
-    )
-    (property "Datasheet" "http://ww1.microchip.com/downloads/en/DeviceDoc/22053C.pdf" (id 3) (at 146.05 82.55 0)
-      (effects (font (size 1.27 1.27)) hide)
-    )
-    (pin "1")
-    (pin "2")
-    (pin "3")
-    (pin "4")
-    (pin "5")
-  )
-  (sheet_instances
-    (path "/" (page "1"))
-  )
-  (symbol_instances
-    (path "/070425be-5ccb-4e88-8c4c-e4baef794b8e"
-      (reference "#PWR?") (unit 1) (value "+3V3") (footprint "")
-    )
-    (path "/3fa75c28-cd45-4a64-8a75-f1e20f7b02e4"
-      (reference "#PWR?") (unit 1) (value "+3V3") (footprint "")
-    )
-    (path "/44d6556c-3980-4535-91e7-ca0f03731d28"
-      (reference "#PWR?") (unit 1) (value "+5V") (footprint "")
-    )
-    (path "/52992af0-bfca-4eff-8f47-ab566d86e29d"
-      (reference "#PWR?") (unit 1) (value "GND") (footprint "")
-    )
-    (path "/d7482a1f-d519-46fd-95ed-f3094f05d90f"
-      (reference "#PWR?") (unit 1) (value "GND") (footprint "")
-    )
-    (path "/96102620-adf7-478e-bad6-78de1078c047"
-      (reference "C?") (unit 1) (value "1uF") (footprint "")
-    )
-    (path "/bcc8b894-fc6c-4a02-b892-9bb6d6a25acb"
-      (reference "C?") (unit 1) (value "1uF") (footprint "")
-    )
-    (path "/0220e075-d97f-4076-83a4-7e5c155e204a"
-      (reference "D?") (unit 1) (value "LED") (footprint "")
-    )
-    (path "/56bc323f-2c11-45f4-9795-9e890654428f"
-      (reference "R?") (unit 1) (value "1k") (footprint "")
-    )
-    (path "/eebe5061-3b92-49eb-a209-d76d8334c777"
-      (reference "U?") (unit 1) (value "BU33SD5WG-TR") (footprint "Package_TO_SOT_SMD:SOT-23-5")
-    )
-  )
 )
