File: hardware/microProc/IO_Connectors.kicad_sch (KiCad schematic)
At the start: 0 parts

Commit message: IO Connector
Parts:
- added J?: POWER, symbol Connector_Generic:Conn_01x02
- added J?: OUTPUT, symbol Connector_Generic:Conn_01x02
- added J?: INPUT, symbol Connector_Generic:Conn_01x02
Connections:
- new net +5V: J?.1 (Pin_1)
- new net ADC_IN1: J?.1 (Pin_1)
- new net DAC_OUT: J?.1 (Pin_1)
- new net GND: J?.2 (Pin_2), J?.2 (Pin_2), J?.2 (Pin_2)
Changed lines of the file:
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@@
 (kicad_sch (version 20211123) (generator eeschema)
   (paper "A4")
+  (junction (at 128.27 90.17) (diameter 0) (color 0 0 0 0)
+  )
+  (wire (pts (xy 128.27 90.17) (xy 147.32 90.17))
+    (stroke (width 0) (type default) (color 0 0 0 0))
+  )
+  (wire (pts (xy 129.54 80.01) (xy 129.54 78.74))
+    (stroke (width 0) (type default) (color 0 0 0 0))
+  )
+  (wire (pts (xy 124.46 82.55) (xy 134.62 82.55))
+    (stroke (width 0) (type default) (color 0 0 0 0))
+  )
+  (wire (pts (xy 147.32 90.17) (xy 147.32 93.98))
+    (stroke (width 0) (type default) (color 0 0 0 0))
+  )
+  (wire (pts (xy 125.73 100.33) (xy 128.27 100.33))
+    (stroke (width 0) (type default) (color 0 0 0 0))
+  )
+  (wire (pts (xy 124.46 80.01) (xy 129.54 80.01))
+    (stroke (width 0) (type default) (color 0 0 0 0))
+  )
+  (wire (pts (xy 128.27 100.33) (xy 128.27 90.17))
+    (stroke (width 0) (type default) (color 0 0 0 0))
+  )
+  (wire (pts (xy 147.32 96.52) (xy 153.67 96.52))
+    (stroke (width 0) (type default) (color 0 0 0 0))
+  )
+  (wire (pts (xy 125.73 102.87) (xy 129.54 102.87))
+    (stroke (width 0) (type default) (color 0 0 0 0))
+  )
+  (global_label "DAC_OUT" (shape input) (at 153.67 96.52 0) (fields_autoplaced)
+    (effects (font (size 1.27 1.27)) (justify left))
+    (property "Intersheet References" "${INTERSHEET_REFS}" (id 0) (at 164.3079 96.4406 0)
+      (effects (font (size 1.27 1.27)) (justify left) hide)
+    )
+  )
+  (global_label "ADC_IN1" (shape input) (at 129.54 102.87 0) (fields_autoplaced)
+    (effects (font (size 1.27 1.27)) (justify left))
+    (property "Intersheet References" "${INTERSHEET_REFS}" (id 0) (at 139.6941 102.7906 0)
+      (effects (font (size 1.27 1.27)) (justify left) hide)
+    )
+  )
+  (symbol (lib_id "Connector_Generic:Conn_01x02") (at 119.38 82.55 180) (unit 1)
+    (in_bom yes) (on_board yes) (fields_autoplaced)
+    (property "Reference" "J?" (id 0) (at 119.38 73.66 0))
+    (property "Value" "POWER" (id 1) (at 119.38 76.2 0))
+    (property "Footprint" "" (id 2) (at 119.38 82.55 0)
+      (effects (font (size 1.27 1.27)) hide)
+    )
+    (property "Datasheet" "~" (id 3) (at 119.38 82.55 0)
+      (effects (font (size 1.27 1.27)) hide)
+    )
+    (pin "1")
+    (pin "2")
+  )
+  (symbol (lib_id "power:GND") (at 128.27 90.17 270) (unit 1)
+    (in_bom yes) (on_board yes) (fields_autoplaced)
+    (property "Reference" "#PWR?" (id 0) (at 121.92 90.17 0)
+      (effects (font (size 1.27 1.27)) hide)
+    )
+    (property "Value" "GND" (id 1) (at 124.46 90.1699 90)
+      (effects (font (size 1.27 1.27)) (justify right))
+    )
+    (property "Footprint" "" (id 2) (at 128.27 90.17 0)
+      (effects (font (size 1.27 1.27)) hide)
+    )
+    (property "Datasheet" "" (id 3) (at 128.27 90.17 0)
+      (effects (font (size 1.27 1.27)) hide)
+    )
+    (pin "1")
+  )
+  (symbol (lib_id "Connector_Generic:Conn_01x02") (at 142.24 96.52 180) (unit 1)
+    (in_bom yes) (on_board yes)
+    (property "Reference" "J?" (id 0) (at 146.05 85.09 0))
+    (property "Value" "OUTPUT" (id 1) (at 146.05 87.63 0))
+    (property "Footprint" "" (id 2) (at 142.24 96.52 0)
+      (effects (font (size 1.27 1.27)) hide)
+    )
+    (property "Datasheet" "~" (id 3) (at 142.24 96.52 0)
+      (effects (font (size 1.27 1.27)) hide)
+    )
+    (pin "1")
+    (pin "2")
+  )
+  (symbol (lib_id "power:+5V") (at 134.62 82.55 0) (unit 1)
+    (in_bom yes) (on_board yes) (fields_autoplaced)
+    (property "Reference" "#PWR?" (id 0) (at 134.62 86.36 0)
+      (effects (font (size 1.27 1.27)) hide)
+    )
+    (property "Value" "+5V" (id 1) (at 134.62 77.47 0))
+    (property "Footprint" "" (id 2) (at 134.62 82.55 0)
+      (effects (font (size 1.27 1.27)) hide)
+    )
+    (property "Datasheet" "" (id 3) (at 134.62 82.55 0)
+      (effects (font (size 1.27 1.27)) hide)
+    )
+    (pin "1")
+  )
+  (symbol (lib_id "power:GND") (at 129.54 78.74 180) (unit 1)
+    (in_bom yes) (on_board yes) (fields_autoplaced)
+    (property "Reference" "#PWR?" (id 0) (at 129.54 72.39 0)
+      (effects (font (size 1.27 1.27)) hide)
+    )
+    (property "Value" "GND" (id 1) (at 129.54 73.66 0))
+    (property "Footprint" "" (id 2) (at 129.54 78.74 0)
+      (effects (font (size 1.27 1.27)) hide)
+    )
+    (property "Datasheet" "" (id 3) (at 129.54 78.74 0)
+      (effects (font (size 1.27 1.27)) hide)
+    )
+    (pin "1")
+  )
+  (symbol (lib_id "Connector_Generic:Conn_01x02") (at 120.65 102.87 180) (unit 1)
+    (in_bom yes) (on_board yes) (fields_autoplaced)
+    (property "Reference" "J?" (id 0) (at 120.65 93.98 0))
+    (property "Value" "INPUT" (id 1) (at 120.65 96.52 0))
+    (property "Footprint" "" (id 2) (at 120.65 102.87 0)
+      (effects (font (size 1.27 1.27)) hide)
+    )
+    (property "Datasheet" "~" (id 3) (at 120.65 102.87 0)
+      (effects (font (size 1.27 1.27)) hide)
+    )
+    (pin "1")
+    (pin "2")
+  )
 )

Commit message: ERC verified, no error
Parts:
- gave numbers to parts that had none: 3
Changed lines of the file:
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@@
   (symbol (lib_id "Connector_Generic:Conn_01x02") (at 119.38 82.55 180) (unit 1)
     (in_bom yes) (on_board yes) (fields_autoplaced)
-    (property "Reference" "J?" (id 0) (at 119.38 73.66 0))
+    (property "Reference" "J1" (id 0) (at 119.38 73.66 0))
     (property "Value" "POWER" (id 1) (at 119.38 76.2 0))
     (property "Footprint" "" (id 2) (at 119.38 82.55 0)
@@
   (symbol (lib_id "power:GND") (at 128.27 90.17 270) (unit 1)
     (in_bom yes) (on_board yes) (fields_autoplaced)
-    (property "Reference" "#PWR?" (id 0) (at 121.92 90.17 0)
+    (property "Reference" "#PWR020" (id 0) (at 121.92 90.17 0)
       (effects (font (size 1.27 1.27)) hide)
     )
@@
   (symbol (lib_id "Connector_Generic:Conn_01x02") (at 142.24 96.52 180) (unit 1)
     (in_bom yes) (on_board yes)
-    (property "Reference" "J?" (id 0) (at 146.05 85.09 0))
+    (property "Reference" "J3" (id 0) (at 146.05 85.09 0))
     (property "Value" "OUTPUT" (id 1) (at 146.05 87.63 0))
     (property "Footprint" "" (id 2) (at 142.24 96.52 0)
@@
   (symbol (lib_id "power:+5V") (at 134.62 82.55 0) (unit 1)
     (in_bom yes) (on_board yes) (fields_autoplaced)
-    (property "Reference" "#PWR?" (id 0) (at 134.62 86.36 0)
+    (property "Reference" "#PWR022" (id 0) (at 134.62 86.36 0)
       (effects (font (size 1.27 1.27)) hide)
     )
@@
   (symbol (lib_id "power:GND") (at 129.54 78.74 180) (unit 1)
     (in_bom yes) (on_board yes) (fields_autoplaced)
-    (property "Reference" "#PWR?" (id 0) (at 129.54 72.39 0)
+    (property "Reference" "#PWR021" (id 0) (at 129.54 72.39 0)
       (effects (font (size 1.27 1.27)) hide)
     )
@@
   (symbol (lib_id "Connector_Generic:Conn_01x02") (at 120.65 102.87 180) (unit 1)
     (in_bom yes) (on_board yes) (fields_autoplaced)
-    (property "Reference" "J?" (id 0) (at 120.65 93.98 0))
+    (property "Reference" "J2" (id 0) (at 120.65 93.98 0))
     (property "Value" "INPUT" (id 1) (at 120.65 96.52 0))
     (property "Footprint" "" (id 2) (at 120.65 102.87 0)

Commit message: Assigning Footprints
Parts:
- J1, J2, J3: footprint (none) -> Connector_JST:JST_XH_B2B-XH-A_1x02_P2.50mm_Vertical
Changed lines of the file:
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@@
     (property "Reference" "J1" (id 0) (at 119.38 73.66 0))
     (property "Value" "POWER" (id 1) (at 119.38 76.2 0))
-    (property "Footprint" "" (id 2) (at 119.38 82.55 0)
+    (property "Footprint" "Connector_JST:JST_XH_B2B-XH-A_1x02_P2.50mm_Vertical" (id 2) (at 119.38 82.55 0)
       (effects (font (size 1.27 1.27)) hide)
     )
@@
     (property "Reference" "J3" (id 0) (at 146.05 85.09 0))
     (property "Value" "OUTPUT" (id 1) (at 146.05 87.63 0))
-    (property "Footprint" "" (id 2) (at 142.24 96.52 0)
+    (property "Footprint" "Connector_JST:JST_XH_B2B-XH-A_1x02_P2.50mm_Vertical" (id 2) (at 142.24 96.52 0)
       (effects (font (size 1.27 1.27)) hide)
     )
@@
     (property "Reference" "J2" (id 0) (at 120.65 93.98 0))
     (property "Value" "INPUT" (id 1) (at 120.65 96.52 0))
-    (property "Footprint" "" (id 2) (at 120.65 102.87 0)
+    (property "Footprint" "Connector_JST:JST_XH_B2B-XH-A_1x02_P2.50mm_Vertical" (id 2) (at 120.65 102.87 0)
       (effects (font (size 1.27 1.27)) hide)
     )
