File: hardware/microProc/STM32_Microcontroller.kicad_sch (KiCad schematic)
At the start: 1 part

Commit message: Séparation des feuilles Kicad
Signed-off-by: Martin RYS <martinrys@sfr.fr>
Parts:
- removed U?: STM32L021K4Tx, Package_QFP:LQFP-32_7x7mm_P0.8mm, symbol MCU_ST_STM32L0:STM32L021K4Tx
- added U?: STM32L021K4Tx, Package_QFP:LQFP-32_7x7mm_P0.8mm, symbol MCU_ST_STM32L0:STM32L021K4Tx
Connections:
- net +3.3V: now also U?.1 (VDD), U?.17 (VDD)
- net +3.3VA: now also U?.5 (VDDA)
- net GND: now also U?.16 (VSS), U?.32 (VSS)
- net NRST: now also U?.4 (NRST)
- net SWCLK: now also U?.24 (PA14)
- net SWDIO: now also U?.23 (PA13)
- net USART2_RX: now also U?.6 (PA0)
- net USUART2_TX: now also U?.8 (PA2)
- new net ADC_IN1: U?.7 (PA1)
- new net DAC_nCS: U?.10 (PA4)
- new net DAC_nLDAC: U?.9 (PA3)
- new net LED_STATUS: U?.18 (PA8)
- new net SPI1_MOSI: U?.13 (PA7)
- new net SPI1_SCK: U?.11 (PA5)

Commit message: KICAD component ST32 microP
Parts:
- added C? (x3): 100n, symbol Device:C
- added C?: 10n, symbol Device:C
- added C?: 4u7, symbol Device:C
- added C?: 1u, symbol Device:C
- added D?: DIODE, symbol pspice:DIODE
- added L?: 39n, symbol Device:L
- added R?: 100k, symbol Device:R
- added R?: 1k, symbol Device:R
Connections:
- net +3.3V: now also C?.1, C?.1, C?.1, L?.2
- net +3.3VA: now also C?.1, C?.1, L?.1
- net GND: now also C?.2, C?.2, C?.2, C?.2, R?.2, R?.2
- net LED_STATUS: now also D?.1 (K)
- net NRST: now also C?.1
- net at U?.31 (PB9): now also R?.1
- new net: C?.2, C?.2
- new net: D?.2 (A), R?.1
- no-connect marks 0 -> 1

Commit message: ERC verified, no error
Parts:
- gave numbers to parts that had none: 11
Connections:
- net SWCLK renamed SWDCK
- net USUART2_TX renamed USART2_TX
- no-connect marks 1 -> 15
Changed lines of the file:
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@@
   (junction (at 66.04 41.91) (diameter 0) (color 0 0 0 0)
   )
-  (no_connect (at 266.7 64.77))
+  (no_connect (at 123.19 88.9))
+  (no_connect (at 123.19 109.22))
+  (no_connect (at 123.19 99.06))
+  (no_connect (at 123.19 96.52))
+  (no_connect (at 148.59 101.6))
+  (no_connect (at 148.59 104.14))
+  (no_connect (at 123.19 104.14))
+  (no_connect (at 148.59 106.68))
+  (no_connect (at 123.19 91.44))
+  (no_connect (at 148.59 91.44))
+  (no_connect (at 148.59 114.3))
+  (no_connect (at 123.19 106.68))
+  (no_connect (at 148.59 99.06))
+  (no_connect (at 123.19 111.76))
+  (no_connect (at 123.19 101.6))
   (wire (pts (xy 135.89 121.92) (xy 135.89 120.65))
     (stroke (width 0) (type default) (color 0 0 0 0))
@@
     )
   )
-  (global_label "USUART2_TX" (shape input) (at 148.59 81.28 0) (fields_autoplaced)
-    (effects (font (size 1.27 1.27)) (justify left))
-    (property "Intersheet References" "${INTERSHEET_REFS}" (id 0) (at 162.5541 81.2006 0)
+  (global_label "USART2_TX" (shape input) (at 148.59 81.28 0) (fields_autoplaced)
+    (effects (font (size 1.27 1.27)) (justify left))
+    (property "Intersheet References" "${INTERSHEET_REFS}" (id 0) (at 161.2236 81.2006 0)
       (effects (font (size 1.27 1.27)) (justify left) hide)
     )
@@
     )
   )
-  (global_label "SWCLK" (shape input) (at 148.59 111.76 0) (fields_autoplaced)
-    (effects (font (size 1.27 1.27)) (justify left))
-    (property "Intersheet References" "${INTERSHEET_REFS}" (id 0) (at 157.2321 111.6806 0)
+  (global_label "SWDCK" (shape input) (at 148.59 111.76 0) (fields_autoplaced)
+    (effects (font (size 1.27 1.27)) (justify left))
+    (property "Intersheet References" "${INTERSHEET_REFS}" (id 0) (at 157.4741 111.6806 0)
       (effects (font (size 1.27 1.27)) (justify left) hide)
     )
@@
   (symbol (lib_id "power:GND") (at 123.19 121.92 0) (unit 1)
     (in_bom yes) (on_board yes) (fields_autoplaced)
-    (property "Reference" "#PWR?" (id 0) (at 123.19 128.27 0)
+    (property "Reference" "#PWR05" (id 0) (at 123.19 128.27 0)
       (effects (font (size 1.27 1.27)) hide)
     )
@@
   (symbol (lib_id "power:+3.3V") (at 133.35 71.12 0) (unit 1)
     (in_bom yes) (on_board yes)
-    (property "Reference" "#PWR?" (id 0) (at 133.35 74.93 0)
+    (property "Reference" "#PWR07" (id 0) (at 133.35 74.93 0)
       (effects (font (size 1.27 1.27)) hide)
     )
@@
   (symbol (lib_id "MCU_ST_STM32L0:STM32L021K4Tx") (at 135.89 93.98 0) (unit 1)
     (in_bom yes) (on_board yes) (fields_autoplaced)
-    (property "Reference" "U?" (id 0) (at 137.9094 119.38 0)
+    (property "Reference" "U1" (id 0) (at 137.9094 119.38 0)
       (effects (font (size 1.27 1.27)) (justify left))
     )
@@
   (symbol (lib_id "Device:R") (at 123.19 118.11 0) (unit 1)
     (in_bom yes) (on_board yes) (fields_autoplaced)
-    (property "Reference" "R?" (id 0) (at 125.73 116.8399 0)
+    (property "Reference" "R2" (id 0) (at 125.73 116.8399 0)
       (effects (font (size 1.27 1.27)) (justify left))
     )
@@
   (symbol (lib_id "Device:C") (at 120.65 80.01 0) (unit 1)
     (in_bom yes) (on_board yes) (fields_autoplaced)
-    (property "Reference" "C?" (id 0) (at 124.46 78.7399 0)
+    (property "Reference" "C4" (id 0) (at 124.46 78.7399 0)
       (effects (font (size 1.27 1.27)) (justify left))
     )
@@
   (symbol (lib_id "power:+3.3VA") (at 154.94 29.21 0) (unit 1)
     (in_bom yes) (on_board yes) (fields_autoplaced)
-    (property "Reference" "#PWR?" (id 0) (at 154.94 33.02 0)
+    (property "Reference" "#PWR010" (id 0) (at 154.94 33.02 0)
       (effects (font (size 1.27 1.27)) hide)
     )
@@
   (symbol (lib_id "power:GND") (at 120.65 83.82 0) (unit 1)
     (in_bom yes) (on_board yes) (fields_autoplaced)
-    (property "Reference" "#PWR?" (id 0) (at 120.65 90.17 0)
+    (property "Reference" "#PWR04" (id 0) (at 120.65 90.17 0)
       (effects (font (size 1.27 1.27)) hide)
     )
@@
   (symbol (lib_id "power:+3.3VA") (at 138.43 71.12 0) (unit 1)
     (in_bom yes) (on_board yes) (fields_autoplaced)
-    (property "Reference" "#PWR?" (id 0) (at 138.43 74.93 0)
+    (property "Reference" "#PWR09" (id 0) (at 138.43 74.93 0)
       (effects (font (size 1.27 1.27)) hide)
     )
@@
   (symbol (lib_id "Device:C") (at 156.21 40.64 0) (unit 1)
     (in_bom yes) (on_board yes) (fields_autoplaced)
-    (property "Reference" "C?" (id 0) (at 160.02 39.3699 0)
+    (property "Reference" "C6" (id 0) (at 160.02 39.3699 0)
       (effects (font (size 1.27 1.27)) (justify left))
     )
@@
   (symbol (lib_id "power:GND") (at 68.58 54.61 0) (unit 1)
     (in_bom yes) (on_board yes) (fields_autoplaced)
-    (property "Reference" "#PWR?" (id 0) (at 68.58 60.96 0)
+    (property "Reference" "#PWR03" (id 0) (at 68.58 60.96 0)
       (effects (font (size 1.27 1.27)) hide)
     )
@@
   (symbol (lib_id "Device:C") (at 74.93 45.72 0) (unit 1)
     (in_bom yes) (on_board yes) (fields_autoplaced)
-    (property "Reference" "C?" (id 0) (at 78.74 44.4499 0)
+    (property "Reference" "C2" (id 0) (at 78.74 44.4499 0)
       (effects (font (size 1.27 1.27)) (justify left))
     )
@@
   (symbol (lib_id "power:+3.3V") (at 132.08 20.32 0) (unit 1)
     (in_bom yes) (on_board yes)
-    (property "Reference" "#PWR?" (id 0) (at 132.08 24.13 0)
+    (property "Reference" "#PWR06" (id 0) (at 132.08 24.13 0)
       (effects (font (size 1.27 1.27)) hide)
     )
@@
   (symbol (lib_id "Device:R") (at 57.15 123.19 0) (unit 1)
     (in_bom yes) (on_board yes) (fields_autoplaced)
-    (property "Reference" "R?" (id 0) (at 59.69 121.9199 0)
+    (property "Reference" "R1" (id 0) (at 59.69 121.9199 0)
       (effects (font (size 1.27 1.27)) (justify left))
     )
@@
   (symbol (lib_id "Device:C") (at 91.44 45.72 0) (unit 1)
     (in_bom yes) (on_board yes) (fields_autoplaced)
-    (property "Reference" "C?" (id 0) (at 95.25 44.4499 0)
+    (property "Reference" "C3" (id 0) (at 95.25 44.4499 0)
       (effects (font (size 1.27 1.27)) (justify left))
     )
@@
   (symbol (lib_id "Device:C") (at 60.96 45.72 0) (unit 1)
     (in_bom yes) (on_board yes) (fields_autoplaced)
-    (property "Reference" "C?" (id 0) (at 64.77 44.4499 0)
+    (property "Reference" "C1" (id 0) (at 64.77 44.4499 0)
       (effects (font (size 1.27 1.27)) (justify left))
     )
@@
   (symbol (lib_id "power:GND") (at 64.77 127 0) (unit 1)
     (in_bom yes) (on_board yes) (fields_autoplaced)
-    (property "Reference" "#PWR?" (id 0) (at 64.77 133.35 0)
+    (property "Reference" "#PWR01" (id 0) (at 64.77 133.35 0)
       (effects (font (size 1.27 1.27)) hide)
     )
@@
   (symbol (lib_id "power:GND") (at 135.89 121.92 0) (unit 1)
     (in_bom yes) (on_board yes) (fields_autoplaced)
-    (property "Reference" "#PWR?" (id 0) (at 135.89 128.27 0)
+    (property "Reference" "#PWR08" (id 0) (at 135.89 128.27 0)
       (effects (font (size 1.27 1.27)) hide)
     )
@@
   (symbol (lib_id "power:+3.3V") (at 66.04 36.83 0) (unit 1)
     (in_bom yes) (on_board yes)
-    (property "Reference" "#PWR?" (id 0) (at 66.04 40.64 0)
+    (property "Reference" "#PWR02" (id 0) (at 66.04 40.64 0)
       (effects (font (size 1.27 1.27)) hide)
     )
@@
   (symbol (lib_id "pspice:DIODE") (at 64.77 114.3 270) (unit 1)
     (in_bom yes) (on_board yes) (fields_autoplaced)
-    (property "Reference" "D?" (id 0) (at 68.58 113.0299 90)
+    (property "Reference" "D1" (id 0) (at 68.58 113.0299 90)
       (effects (font (size 1.27 1.27)) (justify left))
     )
@@
   (symbol (lib_id "Device:C") (at 138.43 40.64 0) (unit 1)
     (in_bom yes) (on_board yes) (fields_autoplaced)
-    (property "Reference" "C?" (id 0) (at 142.24 39.3699 0)
+    (property "Reference" "C5" (id 0) (at 142.24 39.3699 0)
       (effects (font (size 1.27 1.27)) (justify left))
     )
@@
   (symbol (lib_id "Device:L") (at 132.08 29.21 180) (unit 1)
     (in_bom yes) (on_board yes) (fields_autoplaced)
-    (property "Reference" "L?" (id 0) (at 133.35 27.9399 0)
+    (property "Reference" "L1" (id 0) (at 133.35 27.9399 0)
       (effects (font (size 1.27 1.27)) (justify right))
     )

Commit message: Assigning Footprints
Parts:
- C1, C2, C3, C4, C5, C6: footprint (none) -> Capacitor_SMD:C_0805_2012Metric_Pad1.18x1.45mm_HandSolder
- D1: footprint (none) -> LED_SMD:LED_0603_1608Metric_Pad1.05x0.95mm_HandSolder
- L1: footprint (none) -> Inductor_SMD:L_0805_2012Metric_Pad1.05x1.20mm_HandSolder
- R1, R2: footprint (none) -> Resistor_SMD:R_0805_2012Metric_Pad1.20x1.40mm_HandSolder
Changed lines of the file:
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@@
       (effects (font (size 1.27 1.27)) (justify right) hide)
     )
-    (property "Datasheet" "http://www.st.com/st-web-ui/static/active/en/resource/technical/document/datasheet/DM00206858.pdf" (id 3) (at 135.89 93.98 0)
+    (property "Datasheet" "" (id 3) (at 135.89 93.98 0)
       (effects (font (size 1.27 1.27)) hide)
     )
@@
       (effects (font (size 1.27 1.27)) (justify left))
     )
-    (property "Footprint" "" (id 2) (at 121.412 118.11 90)
+    (property "Footprint" "Resistor_SMD:R_0805_2012Metric_Pad1.20x1.40mm_HandSolder" (id 2) (at 121.412 118.11 90)
       (effects (font (size 1.27 1.27)) hide)
     )
@@
       (effects (font (size 1.27 1.27)) (justify left))
     )
-    (property "Footprint" "" (id 2) (at 121.6152 83.82 0)
+    (property "Footprint" "Capacitor_SMD:C_0805_2012Metric_Pad1.18x1.45mm_HandSolder" (id 2) (at 121.6152 83.82 0)
       (effects (font (size 1.27 1.27)) hide)
     )
@@
       (effects (font (size 1.27 1.27)) (justify left))
     )
-    (property "Footprint" "" (id 2) (at 157.1752 44.45 0)
+    (property "Footprint" "Capacitor_SMD:C_0805_2012Metric_Pad1.18x1.45mm_HandSolder" (id 2) (at 157.1752 44.45 0)
       (effects (font (size 1.27 1.27)) hide)
     )
@@
       (effects (font (size 1.27 1.27)) (justify left))
     )
-    (property "Footprint" "" (id 2) (at 75.8952 49.53 0)
+    (property "Footprint" "Capacitor_SMD:C_0805_2012Metric_Pad1.18x1.45mm_HandSolder" (id 2) (at 75.8952 49.53 0)
       (effects (font (size 1.27 1.27)) hide)
     )
@@
       (effects (font (size 1.27 1.27)) (justify left))
     )
-    (property "Footprint" "" (id 2) (at 55.372 123.19 90)
+    (property "Footprint" "Resistor_SMD:R_0805_2012Metric_Pad1.20x1.40mm_HandSolder" (id 2) (at 55.372 123.19 90)
       (effects (font (size 1.27 1.27)) hide)
     )
@@
       (effects (font (size 1.27 1.27)) (justify left))
     )
-    (property "Footprint" "" (id 2) (at 92.4052 49.53 0)
+    (property "Footprint" "Capacitor_SMD:C_0805_2012Metric_Pad1.18x1.45mm_HandSolder" (id 2) (at 92.4052 49.53 0)
       (effects (font (size 1.27 1.27)) hide)
     )
@@
       (effects (font (size 1.27 1.27)) (justify left))
     )
-    (property "Footprint" "" (id 2) (at 61.9252 49.53 0)
+    (property "Footprint" "Capacitor_SMD:C_0805_2012Metric_Pad1.18x1.45mm_HandSolder" (id 2) (at 61.9252 49.53 0)
       (effects (font (size 1.27 1.27)) hide)
     )
@@
       (effects (font (size 1.27 1.27)) (justify left))
     )
-    (property "Footprint" "" (id 2) (at 64.77 114.3 0)
+    (property "Footprint" "LED_SMD:LED_0603_1608Metric_Pad1.05x0.95mm_HandSolder" (id 2) (at 64.77 114.3 0)
       (effects (font (size 1.27 1.27)) hide)
     )
@@
       (effects (font (size 1.27 1.27)) (justify left))
     )
-    (property "Footprint" "" (id 2) (at 139.3952 44.45 0)
+    (property "Footprint" "Capacitor_SMD:C_0805_2012Metric_Pad1.18x1.45mm_HandSolder" (id 2) (at 139.3952 44.45 0)
       (effects (font (size 1.27 1.27)) hide)
     )
@@
       (effects (font (size 1.27 1.27)) (justify right))
     )
-    (property "Footprint" "" (id 2) (at 132.08 29.21 0)
-      (effects (font (size 1.27 1.27)) hide)
-    )
+    (property "Footprint" "Inductor_SMD:L_0805_2012Metric_Pad1.05x1.20mm_HandSolder" (id 2) (at 132.08 29.21 0)
+      (effects (font (size 1.27 1.27)) hide)
+    )
