File: hardware/microProc/SWD_Connector.kicad_sch (KiCad schematic)
At the start: 0 parts

Commit message: SWD connector
Parts:
- added J?: Conn_02x07_Odd_Even, symbol Connector_Generic:Conn_02x07_Odd_Even
Connections:
- new net +3.3V: J?.3 (Pin_3)
- new net GND: J?.11 (Pin_11), J?.5 (Pin_5), J?.7 (Pin_7)
- new net NRST: J?.12 (Pin_12)
- new net SWDCK: J?.6 (Pin_6)
- new net SWDIO: J?.4 (Pin_4)
- new net USART2_RX: J?.13 (Pin_13)
- new net USART2_TX: J?.14 (Pin_14)
Changed lines of the file:
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@@
 (kicad_sch (version 20211123) (generator eeschema)
   (paper "A4")
+  (junction (at 132.08 97.79) (diameter 0) (color 0 0 0 0)
+  )
+  (wire (pts (xy 124.46 92.71) (xy 135.89 92.71))
+    (stroke (width 0) (type default) (color 0 0 0 0))
+  )
+  (wire (pts (xy 148.59 92.71) (xy 157.48 92.71))
+    (stroke (width 0) (type default) (color 0 0 0 0))
+  )
+  (wire (pts (xy 148.59 95.25) (xy 157.48 95.25))
+    (stroke (width 0) (type default) (color 0 0 0 0))
+  )
+  (wire (pts (xy 135.89 95.25) (xy 132.08 95.25))
+    (stroke (width 0) (type default) (color 0 0 0 0))
+  )
+  (wire (pts (xy 148.59 102.87) (xy 157.48 102.87))
+    (stroke (width 0) (type default) (color 0 0 0 0))
+  )
+  (wire (pts (xy 148.59 105.41) (xy 157.48 105.41))
+    (stroke (width 0) (type default) (color 0 0 0 0))
+  )
+  (wire (pts (xy 132.08 97.79) (xy 135.89 97.79))
+    (stroke (width 0) (type default) (color 0 0 0 0))
+  )
+  (wire (pts (xy 132.08 97.79) (xy 132.08 102.87))
+    (stroke (width 0) (type default) (color 0 0 0 0))
+  )
+  (wire (pts (xy 132.08 95.25) (xy 132.08 97.79))
+    (stroke (width 0) (type default) (color 0 0 0 0))
+  )
+  (wire (pts (xy 124.46 105.41) (xy 135.89 105.41))
+    (stroke (width 0) (type default) (color 0 0 0 0))
+  )
+  (wire (pts (xy 124.46 97.79) (xy 132.08 97.79))
+    (stroke (width 0) (type default) (color 0 0 0 0))
+  )
+  (wire (pts (xy 132.08 102.87) (xy 135.89 102.87))
+    (stroke (width 0) (type default) (color 0 0 0 0))
+  )
+  (wire (pts (xy 124.46 88.9) (xy 124.46 92.71))
+    (stroke (width 0) (type default) (color 0 0 0 0))
+  )
+  (global_label "USART2_RX" (shape input) (at 124.46 105.41 180) (fields_autoplaced)
+    (effects (font (size 1.27 1.27)) (justify right))
+    (property "Intersheet References" "${INTERSHEET_REFS}" (id 0) (at 111.524 105.3306 0)
+      (effects (font (size 1.27 1.27)) (justify right) hide)
+    )
+  )
+  (global_label "USART2_TX" (shape input) (at 157.48 105.41 0) (fields_autoplaced)
+    (effects (font (size 1.27 1.27)) (justify left))
+    (property "Intersheet References" "${INTERSHEET_REFS}" (id 0) (at 170.1136 105.3306 0)
+      (effects (font (size 1.27 1.27)) (justify left) hide)
+    )
+  )
+  (global_label "SWDIO" (shape input) (at 157.48 92.71 0) (fields_autoplaced)
+    (effects (font (size 1.27 1.27)) (justify left))
+    (property "Intersheet References" "${INTERSHEET_REFS}" (id 0) (at 165.7593 92.6306 0)
+      (effects (font (size 1.27 1.27)) (justify left) hide)
+    )
+  )
+  (global_label "SWDCK" (shape input) (at 157.48 95.25 0) (fields_autoplaced)
+    (effects (font (size 1.27 1.27)) (justify left))
+    (property "Intersheet References" "${INTERSHEET_REFS}" (id 0) (at 166.3641 95.1706 0)
+      (effects (font (size 1.27 1.27)) (justify left) hide)
+    )
+  )
+  (global_label "NRST" (shape input) (at 157.48 102.87 0) (fields_autoplaced)
+    (effects (font (size 1.27 1.27)) (justify left))
+    (property "Intersheet References" "${INTERSHEET_REFS}" (id 0) (at 164.6707 102.7906 0)
+      (effects (font (size 1.27 1.27)) (justify left) hide)
+    )
+  )
+  (symbol (lib_id "Connector_Generic:Conn_02x07_Odd_Even") (at 140.97 97.79 0) (unit 1)
+    (in_bom yes) (on_board yes) (fields_autoplaced)
+    (property "Reference" "J?" (id 0) (at 142.24 83.82 0))
+    (property "Value" "Conn_02x07_Odd_Even" (id 1) (at 142.24 86.36 0))
+    (property "Footprint" "" (id 2) (at 140.97 97.79 0)
+      (effects (font (size 1.27 1.27)) hide)
+    )
+    (property "Datasheet" "~" (id 3) (at 140.97 97.79 0)
+      (effects (font (size 1.27 1.27)) hide)
+    )
+    (pin "1")
+    (pin "10")
+    (pin "11")
+    (pin "12")
+    (pin "13")
+    (pin "14")
+    (pin "2")
+    (pin "3")
+    (pin "4")
+    (pin "5")
+    (pin "6")
+    (pin "7")
+    (pin "8")
+    (pin "9")
+  )
+  (symbol (lib_id "power:GND") (at 124.46 97.79 0) (unit 1)
+    (in_bom yes) (on_board yes) (fields_autoplaced)
+    (property "Reference" "#PWR?" (id 0) (at 124.46 104.14 0)
+      (effects (font (size 1.27 1.27)) hide)
+    )
+    (property "Value" "GND" (id 1) (at 124.46 102.87 0))
+    (property "Footprint" "" (id 2) (at 124.46 97.79 0)
+      (effects (font (size 1.27 1.27)) hide)
+    )
+    (property "Datasheet" "" (id 3) (at 124.46 97.79 0)
+      (effects (font (size 1.27 1.27)) hide)
+    )
+    (pin "1")
+  )
+  (symbol (lib_id "power:+3.3V") (at 124.46 88.9 0) (unit 1)
+    (in_bom yes) (on_board yes) (fields_autoplaced)
+    (property "Reference" "#PWR?" (id 0) (at 124.46 92.71 0)
+      (effects (font (size 1.27 1.27)) hide)
+    )
+    (property "Value" "+3.3V" (id 1) (at 124.46 83.82 0))
+    (property "Footprint" "" (id 2) (at 124.46 88.9 0)
+      (effects (font (size 1.27 1.27)) hide)
+    )
+    (property "Datasheet" "" (id 3) (at 124.46 88.9 0)
+      (effects (font (size 1.27 1.27)) hide)
+    )
+    (pin "1")
+  )
 )

Commit message: ERC verified, no error
Parts:
- gave numbers to parts that had none: 1
Connections:
- no-connect marks 0 -> 5
Changed lines of the file:
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@@
   (junction (at 132.08 97.79) (diameter 0) (color 0 0 0 0)
   )
+  (no_connect (at 135.89 100.33))
+  (no_connect (at 148.59 100.33))
+  (no_connect (at 135.89 90.17))
+  (no_connect (at 148.59 90.17))
+  (no_connect (at 148.59 97.79))
   (wire (pts (xy 124.46 92.71) (xy 135.89 92.71))
     (stroke (width 0) (type default) (color 0 0 0 0))
@@
   (symbol (lib_id "Connector_Generic:Conn_02x07_Odd_Even") (at 140.97 97.79 0) (unit 1)
     (in_bom yes) (on_board yes) (fields_autoplaced)
-    (property "Reference" "J?" (id 0) (at 142.24 83.82 0))
+    (property "Reference" "J4" (id 0) (at 142.24 83.82 0))
     (property "Value" "Conn_02x07_Odd_Even" (id 1) (at 142.24 86.36 0))
     (property "Footprint" "" (id 2) (at 140.97 97.79 0)
@@
   (symbol (lib_id "power:GND") (at 124.46 97.79 0) (unit 1)
     (in_bom yes) (on_board yes) (fields_autoplaced)
-    (property "Reference" "#PWR?" (id 0) (at 124.46 104.14 0)
+    (property "Reference" "#PWR024" (id 0) (at 124.46 104.14 0)
       (effects (font (size 1.27 1.27)) hide)
     )
@@
   (symbol (lib_id "power:+3.3V") (at 124.46 88.9 0) (unit 1)
     (in_bom yes) (on_board yes) (fields_autoplaced)
-    (property "Reference" "#PWR?" (id 0) (at 124.46 92.71 0)
+    (property "Reference" "#PWR023" (id 0) (at 124.46 92.71 0)
       (effects (font (size 1.27 1.27)) hide)
     )

Commit message: Assigning Footprints
Parts:
- J4: footprint (none) -> Connector_PinHeader_1.27mm:PinHeader_2x07_P1.27mm_Vertical_SMD
Changed lines of the file:
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@@
     (property "Reference" "J4" (id 0) (at 142.24 83.82 0))
     (property "Value" "Conn_02x07_Odd_Even" (id 1) (at 142.24 86.36 0))
-    (property "Footprint" "" (id 2) (at 140.97 97.79 0)
+    (property "Footprint" "Connector_PinHeader_1.27mm:PinHeader_2x07_P1.27mm_Vertical_SMD" (id 2) (at 140.97 97.79 0)
       (effects (font (size 1.27 1.27)) hide)
     )
