File: hardware/microProc/microProc.kicad_sch (KiCad schematic)
At the start: 1 part

Commit message: Changement
Connections:
- net +3.3V: now reaches U?.1 (VDD)
- net +3.3V: now also U?.17 (VDD)
- net DAC_nCS: now reaches U?.10 (PA4)
- net SPI1_SCK: now reaches U?.11 (PA5)
- net SPI1_MOSI: now reaches U?.13 (PA7)
- net LED_STATUS: now reaches U?.18 (PA8)
- net SWDIO: now reaches U?.23 (PA13)
- net SWCLK: now reaches U?.24 (PA14)
- net NRST: now reaches U?.4 (NRST)
- net +3.3VA: now reaches U?.5 (VDDA)
- net USART2_RX: now reaches U?.6 (PA0)
- net ADC_IN1: now reaches U?.7 (PA1)
- net USUART2_TX: now reaches U?.8 (PA2)
- net DAC_nLDAC: now reaches U?.9 (PA3)
Changed lines of the file:
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@@
 (kicad_sch (version 20211123) (generator eeschema)
   (paper "A4")
+  (junction (at 120.65 57.15) (diameter 0) (color 0 0 0 0)
+  )
   (junction (at 123.19 106.68) (diameter 0) (color 0 0 0 0)
   )
@@
     (stroke (width 0) (type default) (color 0 0 0 0))
   )
+  (wire (pts (xy 105.41 62.23) (xy 110.49 62.23))
+    (stroke (width 0) (type default) (color 0 0 0 0))
+  )
+  (wire (pts (xy 120.65 57.15) (xy 123.19 57.15))
+    (stroke (width 0) (type default) (color 0 0 0 0))
+  )
   (wire (pts (xy 123.19 106.68) (xy 123.19 105.41))
     (stroke (width 0) (type default) (color 0 0 0 0))
@@
   (wire (pts (xy 123.19 107.95) (xy 123.19 106.68))
     (stroke (width 0) (type default) (color 0 0 0 0))
+  )
+  (global_label "NRST" (shape input) (at 105.41 62.23 180) (fields_autoplaced)
+    (effects (font (size 1.27 1.27)) (justify right))
+    (property "Intersheet References" "${INTERSHEET_REFS}" (id 0) (at 98.2193 62.1506 0)
+      (effects (font (size 1.27 1.27)) (justify right) hide)
+    )
+  )
+  (global_label "LED_STATUS" (shape input) (at 135.89 82.55 0) (fields_autoplaced)
+    (effects (font (size 1.27 1.27)) (justify left))
+    (property "Intersheet References" "${INTERSHEET_REFS}" (id 0) (at 149.4912 82.4706 0)
+      (effects (font (size 1.27 1.27)) (justify left) hide)
+    )
+  )
+  (global_label "SWCLK" (shape input) (at 135.89 97.79 0) (fields_autoplaced)
+    (effects (font (size 1.27 1.27)) (justify left))
+    (property "Intersheet References" "${INTERSHEET_REFS}" (id 0) (at 144.5321 97.7106 0)
+      (effects (font (size 1.27 1.27)) (justify left) hide)
+    )
+  )
+  (global_label "SWDIO" (shape input) (at 135.89 95.25 0) (fields_autoplaced)
+    (effects (font (size 1.27 1.27)) (justify left))
+    (property "Intersheet References" "${INTERSHEET_REFS}" (id 0) (at 144.1693 95.1706 0)
+      (effects (font (size 1.27 1.27)) (justify left) hide)
+    )
+  )
+  (global_label "ADC_IN1" (shape input) (at 135.89 64.77 0) (fields_autoplaced)
+    (effects (font (size 1.27 1.27)) (justify left))
+    (property "Intersheet References" "${INTERSHEET_REFS}" (id 0) (at 146.0441 64.6906 0)
+      (effects (font (size 1.27 1.27)) (justify left) hide)
+    )
+  )
+  (global_label "SPI1_SCK" (shape input) (at 135.89 74.93 0) (fields_autoplaced)
+    (effects (font (size 1.27 1.27)) (justify left))
+    (property "Intersheet References" "${INTERSHEET_REFS}" (id 0) (at 147.3141 74.8506 0)
+      (effects (font (size 1.27 1.27)) (justify left) hide)
+    )
+  )
+  (global_label "DAC_nCS" (shape input) (at 135.89 72.39 0) (fields_autoplaced)
+    (effects (font (size 1.27 1.27)) (justify left))
+    (property "Intersheet References" "${INTERSHEET_REFS}" (id 0) (at 146.5279 72.3106 0)
+      (effects (font (size 1.27 1.27)) (justify left) hide)
+    )
+  )
+  (global_label "DAC_nLDAC" (shape input) (at 135.89 69.85 0) (fields_autoplaced)
+    (effects (font (size 1.27 1.27)) (justify left))
+    (property "Intersheet References" "${INTERSHEET_REFS}" (id 0) (at 148.705 69.7706 0)
+      (effects (font (size 1.27 1.27)) (justify left) hide)
+    )
+  )
+  (global_label "USART2_RX" (shape input) (at 135.89 62.23 0) (fields_autoplaced)
+    (effects (font (size 1.27 1.27)) (justify left))
+    (property "Intersheet References" "${INTERSHEET_REFS}" (id 0) (at 148.826 62.1506 0)
+      (effects (font (size 1.27 1.27)) (justify left) hide)
+    )
+  )
+  (global_label "USUART2_TX" (shape output) (at 135.89 67.31 0) (fields_autoplaced)
+    (effects (font (size 1.27 1.27)) (justify left))
+    (property "Intersheet References" "${INTERSHEET_REFS}" (id 0) (at 149.8541 67.2306 0)
+      (effects (font (size 1.27 1.27)) (justify left) hide)
+    )
+  )
+  (global_label "SPI1_MOSI" (shape input) (at 135.89 80.01 0) (fields_autoplaced)
+    (effects (font (size 1.27 1.27)) (justify left))
+    (property "Intersheet References" "${INTERSHEET_REFS}" (id 0) (at 148.1607 79.9306 0)
+      (effects (font (size 1.27 1.27)) (justify left) hide)
+    )
+  )
+  (symbol (lib_id "power:+3.3VA") (at 125.73 57.15 0) (unit 1)
+    (in_bom yes) (on_board yes) (fields_autoplaced)
+    (property "Reference" "#PWR?" (id 0) (at 125.73 60.96 0)
+      (effects (font (size 1.27 1.27)) hide)
+    )
+    (property "Value" "+3.3VA" (id 1) (at 125.73 52.07 0))
+    (property "Footprint" "" (id 2) (at 125.73 57.15 0)
+      (effects (font (size 1.27 1.27)) hide)
+    )
+    (property "Datasheet" "" (id 3) (at 125.73 57.15 0)
+      (effects (font (size 1.27 1.27)) hide)
+    )
+    (pin "1")
   )
   (symbol (lib_id "power:+5V") (at 171.45 59.69 0) (unit 1)
@@
     )
     (property "Datasheet" "" (id 3) (at 171.45 59.69 0)
+      (effects (font (size 1.27 1.27)) hide)
+    )
+    (pin "1")
+  )
+  (symbol (lib_id "power:+3.3V") (at 120.65 57.15 0) (unit 1)
+    (in_bom yes) (on_board yes)
+    (property "Reference" "#PWR?" (id 0) (at 120.65 60.96 0)
+      (effects (font (size 1.27 1.27)) hide)
+    )
+    (property "Value" "+3.3V" (id 1) (at 119.38 52.07 0))
+    (property "Footprint" "" (id 2) (at 120.65 57.15 0)
+      (effects (font (size 1.27 1.27)) hide)
+    )
+    (property "Datasheet" "" (id 3) (at 120.65 57.15 0)
       (effects (font (size 1.27 1.27)) hide)
     )
@@
   )
   (symbol_instances
+    (path "/3a28413c-eff0-47c5-96bf-e45287297482"
+      (reference "#PWR?") (unit 1) (value "+3.3VA") (footprint "")
+    )
     (path "/5b1b5739-fcf0-4d2e-89c6-69c8e4c74271"
       (reference "#PWR?") (unit 1) (value "+5V") (footprint "")
     )
+    (path "/894c478e-b272-436e-a322-dbff75657972"
+      (reference "#PWR?") (unit 1) (value "+3.3V") (footprint "")
+    )
     (path "/b0c346e6-884e-4682-92ba-11a470e3fd7c"

Commit message: Séparation des feuilles Kicad
Signed-off-by: Martin RYS <martinrys@sfr.fr>
Parts:
- removed U?: STM32L021K4Tx, Package_QFP:LQFP-32_7x7mm_P0.8mm, symbol MCU_ST_STM32L0:STM32L021K4Tx
Other:
- added sheet DAC MCP4801 (DAC_MCP4801.kicad_sch)
- added sheet IO Connectors (IO_Connectors.kicad_sch)
- added sheet Mounting holes (Mounting_holes.kicad_sch)
- added sheet Power supply (Power_supply.kicad_sch)
- added sheet STM32 Microcontroller (STM32_Microcontroller.kicad_sch)
- added sheet SWD Connector (SWD_Connector.kicad_sch)
